File: Arduino_MEGA2560_ref.sch (EAGLE design)
At the start: 74 parts, among them IC1 7805DT, IC2 7805DT, T1 PHT8N06LTSOT223, T2 PHT8N06LTSOT223, T3 PHT8N06LTSOT223, T4 PHT8N06LTSOT223, T5 PHT8N06LTSOT223, T6 PHT8N06LTSOT223, X1 MKDSN1,5/2-5,08, X2 MKDSN1,5/2-5,08, X3 MKDSN1,5/2-5,08, X4 MKDSN1,5/2-5,08, X5 MKDSN1,5/2-5,08, X6 MKDSN1,5/2-5,08, X7 5566-4, X9 MKDSN1,5/2-5,08

Commit message: doing moving
Connections:
- net ADC13: no longer R7.1
- net ADC14: now also R7.1; no longer R11.1
- net ADC15: now also R11.1
Changed lines of the file:
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@@
 <setting verticaltext="up"/>
 </settings>
-<grid distance="0.1" unitdist="inch" unit="inch" style="lines" multiple="1" display="yes" altdistance="0.01" altunitdist="inch" altunit="inch"/>
+<grid distance="0.1" unitdist="inch" unit="inch" style="lines" multiple="1" display="no" altdistance="0.01" altunitdist="inch" altunit="inch"/>
 <layers>
 <layer number="1" name="Top" color="4" fill="1" visible="no" active="no"/>
@@
 <pinref part="ADCH" gate="A" pin="6"/>
 </segment>
+</net>
+<net name="ADC14" class="0">
+<segment>
+<wire x1="104.14" y1="48.26" x2="71.12" y2="48.26" width="0.1524" layer="91"/>
+<label x="76.2" y="48.895" size="1.778" layer="95"/>
+<pinref part="ADCH" gate="A" pin="7"/>
+</segment>
 <segment>
 <pinref part="R7" gate="G$1" pin="1"/>
@@
 </segment>
 </net>
-<net name="ADC14" class="0">
-<segment>
-<wire x1="104.14" y1="48.26" x2="71.12" y2="48.26" width="0.1524" layer="91"/>
-<label x="76.2" y="48.895" size="1.778" layer="95"/>
-<pinref part="ADCH" gate="A" pin="7"/>
+<net name="ADC15" class="0">
+<segment>
+<wire x1="71.12" y1="50.8" x2="104.14" y2="50.8" width="0.1524" layer="91"/>
+<label x="76.2" y="51.435" size="1.778" layer="95"/>
+<pinref part="ADCH" gate="A" pin="8"/>
 </segment>
 <segment>
@@
 </segment>
 </net>
-<net name="ADC15" class="0">
-<segment>
-<wire x1="71.12" y1="50.8" x2="104.14" y2="50.8" width="0.1524" layer="91"/>
-<label x="76.2" y="51.435" size="1.778" layer="95"/>
-<pinref part="ADCH" gate="A" pin="8"/>
-</segment>
-</net>

Commit message: done handmade
Parts:
- added C9: 1uF, resistor:C-EUC0805
- C5: value (none) -> 1uF
Connections:
- removed net N$19: R21.2, X10-1.1
- new net N$22: R21.2, X10-2.1
- net GND: now also C9.2
- net N$18: now also X10-1.1; no longer X10-2.1
- net TXD1/INT3: now also C9.1
Other:
- moved on the sheet: C5, C6, IC2, OC2, R19, R20, X10-1, X10-2, X9-1, X9-2

Commit message: doing factory
Parts:
- removed C7, C8: 1uF, resistor:C-EUC0805
- removed T1, T2, T3, T4, T5, T6: PHT8N06LTSOT223, NFET_transistors:PHT8N06LTSOT223
- removed X10, X11, X12, X13, X14: (no value), con-phoenix-254:MPT2
- added Q1, Q11, Q13, Q3, Q5, Q7, Q9: IRLML2502, NFET_transistors:IRLML2502
- added Q10, Q12, Q14, Q2, Q4, Q6, Q8: PF610BL, NFET_transistors:PF610BL
- added R22: 0, resistor:R-EU_M0805
- added X15, X16: 1751251, con-phoenix-350:1751251
- added X17: 1751264, con-phoenix-350:1751264
- R15: value 10 -> 1K
- R16: value 1K -> 0
- X8: value (none) -> 1751248; device con-phoenix-254:MPT2 -> con-phoenix-350:1751248
Connections:
- net +5V: now also R15.1, X15-2.K, X16-2.K; no longer X11-1.1, X13-2.1
- net GND: now also Q1.S, Q10.S, Q11.S, Q12.S, Q2.S, Q3.S, Q4.S, Q5.S, Q6.S, Q7.S, Q8.S, Q9.S, R16.2, R22.2, X15-1.K, X16-3.K, X17-1.K, X17-2.K; no longer T1.S, T2.S, T3.S, T4.S, T5.S, T6.S, X11-2.1, X13-1.1, X14-1.1, X8-1.1
- net GNDA: now also Q13.S, Q14.S, R22.1; no longer C7.2, C8.2
- net N$1: now also Q11.G, Q12.G; no longer T1.G
- net N$10: now also Q1.D, Q2.D; no longer T5.D
- net N$11: now also Q5.G, Q6.G; no longer T6.G
- net N$12: now also Q5.D, Q6.D; no longer T6.D
- net N$14: now also Q13.D, Q14.D; no longer R16.2
- net N$17: no longer C8.1
- net N$18: now also X8-1.K; no longer X10-1.1
- net N$2: now also Q10.G, Q9.G; no longer T2.G
- net N$21: now also Q13.G, Q14.G; no longer C7.1, R15.1
- net N$22: now also X8-2.K; no longer X10-2.1
- net N$3: now also Q3.G, Q4.G; no longer T4.G
- net N$4: now also Q11.D, Q12.D; no longer T1.D
- net N$5: now also Q7.G, Q8.G; no longer T3.G
- net N$6: now also Q10.D, Q9.D; no longer T2.D
- net N$7: now also Q7.D, Q8.D; no longer T3.D
- net N$8: now also Q3.D, Q4.D; no longer T4.D
- net N$9: now also Q1.G, Q2.G; no longer T5.G
- net PB4: now also X15-3.K; no longer X12-2.1
- net PB6: now also X17-3.K; no longer X14-2.1
- net PB7: now also X17-4.K; no longer X8-2.1
- net PH6: now also X16-1.K; no longer X12-1.1
Other:
- moved on the sheet: C1, C2, C4, D1, D2, D3, D4, D5, D6, L3, L4, PWMH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

Commit message: doiing CAM
Parts:
- removed ICSP: ICSP, pinhead:PINHD-2X3
- added TP1: PTR1TP20SQ, testpad:PTR1TP20SQ
- added X10: MKDSN1,5/2-5,08, con-phoenix-508:MKDSN1,5/2-5,08
Connections:
- net +24V: now also X10-1.KL
- net GND: now also X16-1.K; no longer X16-3.K
- net GNDA: now also X10-2.KL
- net N$21: now also TP1.TP
- net PH6: now also X16-3.K; no longer X16-1.K
Other:
- moved on the sheet: X16-1, X16-3
Changed lines of the file:
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@@
 </classes>
 <parts>
-<part name="ICSP" library="pinhead" deviceset="PINHD-2X3" device="" value="ICSP"/>
 <part name="PWML" library="pinhead" deviceset="PINHD-1X8" device=""/>
 <part name="PWMH" library="pinhead" deviceset="PINHD-1X8" device=""/>
@@
 <part name="R16" library="resistor" deviceset="R-EU_" device="M0805" value="0"/>
 <part name="R22" library="resistor" deviceset="R-EU_" device="M0805" value="0"/>
+<part name="X10" library="con-phoenix-508" deviceset="MKDSN1,5/2-5,08" device=""/>
+<part name="GND1" library="supply1" deviceset="GNDA" device=""/>
+<part name="P+1" library="supply1" deviceset="+24V" device=""/>
+<part name="TP1" library="testpad" deviceset="PTR1" device="TP20SQ" value="PTR1TP20SQ"/>
 </parts>
 <sheets>
@@
 </plain>
 <instances>
-<instance part="ICSP" gate="A" x="281.94" y="152.4"/>
 <instance part="PWML" gate="A" x="233.68" y="38.1" smashed="yes" rot="MR180">
 <attribute name="NAME" x="243.205" y="37.465" size="1.778" layer="95" rot="MR180"/>
@@
 <attribute name="VALUE" x="176.53" y="89.789" size="1.778" layer="96" rot="R180"/>
 </instance>
-<instance part="X16" gate="-1" x="182.88" y="83.82" smashed="yes" rot="R180">
+<instance part="X16" gate="-1" x="238.76" y="88.9" smashed="yes">
+<attribute name="NAME" x="240.03" y="88.011" size="1.778" layer="95"/>
+<attribute name="VALUE" x="245.11" y="90.551" size="1.778" layer="96"/>
+</instance>
+<instance part="X16" gate="-2" x="238.76" y="93.98"/>
+<instance part="X16" gate="-3" x="182.88" y="83.82" smashed="yes" rot="R180">
 <attribute name="NAME" x="181.61" y="84.709" size="1.778" layer="95" rot="R180"/>
 <attribute name="VALUE" x="176.53" y="82.169" size="1.778" layer="96" rot="R180"/>
 </instance>
-<instance part="X16" gate="-2" x="238.76" y="93.98"/>
-<instance part="X16" gate="-3" x="238.76" y="88.9"/>
 <instance part="X17" gate="-1" x="259.08" y="78.74"/>
 <instance part="X17" gate="-2" x="259.08" y="83.82"/>
@@
 <attribute name="VALUE" x="361.95" y="178.562" size="1.778" layer="96" rot="R180"/>
 </instance>
+<instance part="X10" gate="-1" x="274.32" y="208.28" rot="R90"/>
+<instance part="X10" gate="-2" x="279.4" y="208.28" rot="R90"/>
+<instance part="GND1" gate="1" x="279.4" y="200.66"/>
+<instance part="P+1" gate="1" x="269.24" y="210.82" smashed="yes">
+<attribute name="VALUE" x="271.78" y="210.82" size="1.778" layer="96" rot="R90"/>
+</instance>
+<instance part="TP1" gate="G$1" x="218.44" y="160.02" rot="R270"/>
 </instances>
 <busses>
@@
 <wire x1="231.14" y1="88.9" x2="233.68" y2="88.9" width="0.1524" layer="91"/>
 <wire x1="233.68" y1="88.9" x2="233.68" y2="86.36" width="0.1524" layer="91"/>
+<pinref part="X15" gate="-1" pin="K"/>
+<pinref part="X16" gate="-1" pin="K"/>
 <wire x1="233.68" y1="88.9" x2="236.22" y2="88.9" width="0.1524" layer="91"/>
 <junction x="233.68" y="88.9"/>
-<pinref part="X15" gate="-1" pin="K"/>
-<pinref part="X16" gate="-3" pin="K"/>
 </segment>
 <segment>
@@
 <wire x1="185.42" y1="83.82" x2="198.12" y2="83.82" width="0.1524" layer="91"/>
 <pinref part="PWMH" gate="A" pin="2"/>
-<pinref part="X16" gate="-1" pin="K"/>
+<pinref part="X16" gate="-3" pin="K"/>
 </segment>
 </net>
@@
 <pinref part="X9" gate="-1" pin="KL"/>
 </segment>
+<segment>
+<wire x1="274.32" y1="200.66" x2="269.24" y2="200.66" width="0.1524" layer="91"/>
+<pinref part="P+1" gate="1" pin="+24V"/>
+<wire x1="269.24" y1="200.66" x2="269.24" y2="208.28" width="0.1524" layer="91"/>
+<pinref part="X10" gate="-1" pin="KL"/>
+<wire x1="274.32" y1="200.66" x2="274.32" y2="205.74" width="0.1524" layer="91"/>
+</segment>
 </net>
 <net name="GNDA" class="0">
@@
 <wire x1="208.28" y1="162.56" x2="208.28" y2="160.02" width="0.1524" layer="91"/>
 </segment>
+<segment>
+<pinref part="X10" gate="-2" pin="KL"/>
+<pinref part="GND1" gate="1" pin="GNDA"/>
+<wire x1="279.4" y1="205.74" x2="279.4" y2="203.2" width="0.1524" layer="91"/>
+</segment>
 </net>
 <net name="+5V_1" class="0">
@@
 <wire x1="238.76" y1="167.64" x2="238.76" y2="172.72" width="0.1524" layer="91"/>
 <pinref part="Q14" gate="G$1" pin="G"/>
-</segment>
-</net>
+<pinref part="TP1" gate="G$1" pin="TP"/>
+<wire x1="220.98" y1="160.02" x2="223.52" y2="160.02" width="0.1524" layer="91"/>
+<wire x1="223.52" y1="160.02" x2="223.52" y2="167.64" width="0.1524" layer="91"/>
+<junction x="223.52" y="167.64"/>
+</segment>
+</net>

Commit message: Added new Valves controls
Parts:
- added C7: 0.1uF, resistor:C-EUC0805
- added D7, D8: (no value), diode:DIODE-DO214AA
- added Q15, Q17: IRLML2502, NFET_transistors:IRLML2502
- added Q16, Q18: PF610BL, NFET_transistors:PF610BL
- added R23, R24, R26, R28: 1K, resistor:R-EU_M0805
- added R25, R27: 10, resistor:R-EU_M0805
- added X11, X12, X13: 1751251, con-phoenix-350:1751251
- added X14: MKDSN1,5/2-5,08, con-phoenix-508:MKDSN1,5/2-5,08
- X17: value 1751264 -> MKDSN1,5/2-5,08; device con-phoenix-350:1751264 -> con-phoenix-508:MKDSN1,5/2-5,08
Connections:
- removed net PH5: PWMH.1
- new net N$24: Q17.G, Q18.G, R25.2, R26.2
- new net N$25: D7.A, Q17.D, Q18.D, X14-1.KL
- new net N$26: Q15.G, Q16.G, R27.2, R28.2
- new net N$27: D8.A, Q15.D, Q16.D, X17-2.KL
- net +12V: now also D7.C, D8.C, X14-2.KL, X17-1.KL
- net +5V: now also R24.1, X11-2.K; no longer R15.1
- net +5V_1: now also R15.1
- net ADC12: now also R7.1
- net ADC13: now also R11.1
- net ADC14: now also R27.1; no longer R7.1
- net ADC15: now also R25.1; no longer R11.1
- net ADC4: now also R5.1
- net ADC5: no longer R5.1
- net GND: now also C7.2, Q15.S, Q16.S, Q17.S, Q18.S, R26.1, R28.1, X11-1.K, X13-1.K, X13-2.K, X13-3.K; no longer X17-1.K, X17-2.K
- net GNDA: now also R23.2
- net N$18: now also X8-2.K; no longer X8-1.K
- net N$21: now also R23.1
- net N$22: now also X8-1.K; no longer X8-2.K
- net PB5: now also C7.1, R24.2, X12-1.K
- net PB6: now also X12-2.K; no longer X17-3.K
- net PB7: now also X12-3.K; no longer X17-4.K
- net PH4: now also X11-3.K
Other:
- moved on the sheet: X15-3, X16-3, X7-1, X7-2, X8-1, X8-2

Commit message: Done new version - added new valves
Parts:
- X1, X10, X14, X2, X3, X4, X5, X6, X9: value MKDSN1,5/2-5,08 -> MKDSN
Changed lines of the file:
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@@
 <part name="GND2" library="supply1" deviceset="GND" device=""/>
 <part name="D1" library="diode" deviceset="DIODE-" device="DO214AA"/>
-<part name="X1" library="con-phoenix-508" deviceset="MKDSN1,5/2-5,08" device=""/>
+<part name="X1" library="con-phoenix-508" deviceset="MKDSN1,5/2-5,08" device="" value="MKDSN"/>
 <part name="R3" library="resistor" deviceset="R-EU_" device="M0805" value="10"/>
 <part name="R4" library="resistor" deviceset="R-EU_" device="M0805" value="1K"/>
 <part name="GND4" library="supply1" deviceset="GND" device=""/>
 <part name="D2" library="diode" deviceset="DIODE-" device="DO214AA"/>
-<part name="X2" library="con-phoenix-508" deviceset="MKDSN1,5/2-5,08" device=""/>
+<part name="X2" library="con-phoenix-508" deviceset="MKDSN1,5/2-5,08" device="" value="MKDSN"/>
 <part name="R5" library="resistor" deviceset="R-EU_" device="M0805" value="10"/>
 <part name="R6" library="resistor" deviceset="R-EU_" device="M0805" value="1K"/>
 <part name="GND7" library="supply1" deviceset="GND" device=""/>
 <part name="D3" library="diode" deviceset="DIODE-" device="DO214AA"/>
-<part name="X3" library="con-phoenix-508" deviceset="MKDSN1,5/2-5,08" device=""/>
+<part name="X3" library="con-phoenix-508" deviceset="MKDSN1,5/2-5,08" device="" value="MKDSN"/>
 <part name="P+2" library="supply1" deviceset="+12V" device=""/>
 <part name="P+3" library="supply1" deviceset="+12V" device=""/>
@@
 <part name="GND3" library="supply1" deviceset="GND" device=""/>
 <part name="D4" library="diode" deviceset="DIODE-" device="DO214AA"/>
-<part name="X4" library="con-phoenix-508" deviceset="MKDSN1,5/2-5,08" device=""/>
+<part name="X4" library="con-phoenix-508" deviceset="MKDSN1,5/2-5,08" device="" value="MKDSN"/>
 <part name="P+7" library="supply1" deviceset="+12V" device=""/>
 <part name="R9" library="resistor" deviceset="R-EU_" device="M0805" value="10"/>
@@
 <part name="GND6" library="supply1" deviceset="GND" device=""/>
 <part name="D5" library="diode" deviceset="DIODE-" device="DO214AA"/>
-<part name="X5" library="con-phoenix-508" deviceset="MKDSN1,5/2-5,08" device=""/>
+<part name="X5" library="con-phoenix-508" deviceset="MKDSN1,5/2-5,08" device="" value="MKDSN"/>
 <part name="P+8" library="supply1" deviceset="+12V" device=""/>
 <part name="R11" library="resistor" deviceset="R-EU_" device="M0805" value="10"/>
@@
 <part name="GND8" library="supply1" deviceset="GND" device=""/>
 <part name="D6" library="diode" deviceset="DIODE-" device="DO214AA"/>
-<part name="X6" library="con-phoenix-508" deviceset="MKDSN1,5/2-5,08" device=""/>
+<part name="X6" library="con-phoenix-508" deviceset="MKDSN1,5/2-5,08" device="" value="MKDSN"/>
 <part name="P+9" library="supply1" deviceset="+12V" device=""/>
 <part name="X7" library="con-molex" deviceset="5566-4" device=""/>
@@
 <part name="L3" library="inductor-neosid" deviceset="SM-NE45" device=""/>
 <part name="L4" library="inductor-neosid" deviceset="SM-NE45" device=""/>
-<part name="X9" library="con-phoenix-508" deviceset="MKDSN1,5/2-5,08" device=""/>
+<part name="X9" library="con-phoenix-508" deviceset="MKDSN1,5/2-5,08" device="" value="MKDSN"/>
 <part name="C9" library="resistor" deviceset="C-EU" device="C0805" value="1uF"/>
 <part name="Q1" library="NFET_transistors" deviceset="IRLML2502" device=""/>
@@
 <part name="R16" library="resistor" deviceset="R-EU_" device="M0805" value="0"/>
 <part name="R22" library="resistor" deviceset="R-EU_" device="M0805" value="0"/>
-<part name="X10" library="con-phoenix-508" deviceset="MKDSN1,5/2-5,08" device=""/>
+<part name="X10" library="con-phoenix-508" deviceset="MKDSN1,5/2-5,08" device="" value="MKDSN"/>
 <part name="GND1" library="supply1" deviceset="GNDA" device=""/>
 <part name="P+1" library="supply1" deviceset="+24V" device=""/>
@@
 <part name="GND24" library="supply1" deviceset="GND" device=""/>
 <part name="D7" library="diode" deviceset="DIODE-" device="DO214AA"/>
-<part name="X14" library="con-phoenix-508" deviceset="MKDSN1,5/2-5,08" device=""/>
+<part name="X14" library="con-phoenix-508" deviceset="MKDSN1,5/2-5,08" device="" value="MKDSN"/>
 <part name="P+18" library="supply1" deviceset="+12V" device=""/>
 <part name="R27" library="resistor" deviceset="R-EU_" device="M0805" value="10"/>
